File: board/USB-I2C.kicad_pcb (KiCad board)
At the start: 2 copper layers, 44 x 18 mm, 17 parts, among them J1 USB_OTG, J2 Conn_01x06, U1 SPX3819, U2 STM32F042K4Tx, X1 I2C-6P, X2 I2C, X3 SWD

Commit message: WIP
Parts:
- C1, C2, C3, C4, C5: footprint Capacitors_SMD:C_0805 -> Capacitor_SMD:C_0805_2012Metric
- D1: footprint LEDs:LED_0805 -> LED_SMD:LED_0805_2012Metric
- J2: footprint Pin_Headers:Pin_Header_Straight_1x06_Pitch2.54mm -> Connector_PinHeader_2.54mm:PinHeader_1x06_P2.54mm_Vertical
- R1, R2, R3, R4: footprint Resistors_SMD:R_0805 -> Resistor_SMD:R_0805_2012Metric
- U1: footprint TO_SOT_Packages_SMD:TSOT-23-5 -> Package_TO_SOT_SMD:SOT-23-5
- U2: footprint Housings_QFP:LQFP-32_7x7mm_Pitch0.8mm -> Package_QFP:LQFP-32_7x7mm_P0.8mm
Connections:
- J1 pad 4: (no net) -> Net-(J1-Pad4)
- U1 pad 4: (no net) -> Net-(U1-Pad4)
- U2 pad 10: (no net) -> Net-(U2-Pad10)
- U2 pad 11: (no net) -> Net-(U2-Pad11)
- U2 pad 12: (no net) -> Net-(U2-Pad12)
- U2 pad 13: (no net) -> Net-(U2-Pad13)
- U2 pad 14: (no net) -> Net-(U2-Pad14)
- U2 pad 15: (no net) -> Net-(U2-Pad15)
- U2 pad 2: (no net) -> Net-(U2-Pad2)
- U2 pad 25: (no net) -> Net-(U2-Pad25)
- U2 pad 26: (no net) -> Net-(U2-Pad26)
- U2 pad 27: (no net) -> Net-(U2-Pad27)
- U2 pad 28: (no net) -> Net-(U2-Pad28)
- U2 pad 29: (no net) -> Net-(U2-Pad29)
- U2 pad 3: (no net) -> Net-(U2-Pad3)
- U2 pad 6: (no net) -> Net-(U2-Pad6)
- U2 pad 7: (no net) -> Net-(U2-Pad7)
- U2 pad 8: (no net) -> Net-(U2-Pad8)
- U2 pad 9: (no net) -> Net-(U2-Pad9)

Commit message: WIP
Parts:
- J1: footprint device.farm:conn_usb_B_micro_smd-2 -> Drake:conn_usb_B_micro_smd-2
- X1: footprint device.farm:Micro-Match-FOB-6 -> Drake:Micro-Match-FOB-6
- X2: footprint device.farm:Micro-Match-FOB-4 -> Drake:Micro-Match-FOB-4
- X3: footprint device.farm:SWD -> Drake:SWD
Other:
- board text added: "USB-I2C v1.0 CC-BY-SA Drake"
- board text removed: "USB-I2C v1.0 CC-BY-SA DEVICE.FARM"

Commit message: WIP
Parts:
- U2: value STM32F042K4Tx -> ATSAMD11C14A-SS; footprint Package_QFP:LQFP-32_7x7mm_P0.8mm -> Package_SO:SOIC-14_3.9x8.7mm_P1.27mm
- moved U2 1.12 mm to (163.5, 109.0), turned to 180 degrees
Connections:
- R1 pad 1: Net-(R1-Pad1) -> /LED
- U2 pad 1: +3V3 -> /ALERT
- U2 pad 10: Net-(U2-Pad10) -> /USB_DP
- U2 pad 11: Net-(U2-Pad11) -> GND
- U2 pad 12: Net-(U2-Pad12) -> +3V3
- U2 pad 13: Net-(U2-Pad13) -> /LED
- U2 pad 4: Net-(C1-Pad1) -> /SCL
- U2 pad 5: +3V3 -> /SDA
- U2 pad 6: Net-(U2-Pad6) -> Net-(C1-Pad1)
- U2 pad 7: Net-(U2-Pad7) -> /SWCLK
- U2 pad 8: Net-(U2-Pad8) -> /SWDIO
- U2 pad 9: Net-(U2-Pad9) -> /USB_DM
Routing:
- net Net-(C1-Pad1): track 10.2 -> 18.8 mm, vias 2 -> 0
- net GND: track 40.0 -> 32.3 mm
- net /SCL: track 60.3 -> 54.0 mm
- net /LED: track 0.00 -> 4.35 mm
- net /USB_DP: track 13.6 -> 9.55 mm
- net /USB_DM: track 13.4 -> 9.52 mm
- net Net-(R1-Pad1): track 2.93 -> 0.00 mm
- net /SDA: track 45.7 -> 43.0 mm
- net /SWCLK: track 6.79 -> 9.41 mm, vias 2 -> 1
- net /SWDIO: track 8.27 -> 7.23 mm, vias 2 -> 0
- net /ALERT: track 38.7 -> 39.3 mm, vias 3 -> 1
Other:
- outline, holes or cut-outs redrawn
- board text added: "USB-I2C v1.1 CC-BY-SA drake.cz"
- board text removed: "USB-I2C v1.0 CC-BY-SA Drake"
