File: board/USB-I2C.sch (KiCad schematic (older format))
At the start: 17 parts, among them J1 USB_OTG, J2 Conn_01x06, U1 SPX3819, U2 STM32F042K4Tx, X1 I2C-6P, X2 I2C, X3 SWD

Commit message: WIP
Parts:
- C1, C2, C3, C4, C5: footprint Capacitors_SMD:C_0805 -> Capacitor_SMD:C_0805_2012Metric; symbol C -> Device:C
- D1: footprint LEDs:LED_0805 -> LED_SMD:LED_0805_2012Metric; symbol LED -> Device:LED
- J1: symbol USB_OTG -> Connector:USB_OTG
- J2: footprint Pin_Headers:Pin_Header_Straight_1x06_Pitch2.54mm -> Connector_PinHeader_2.54mm:PinHeader_1x06_P2.54mm_Vertical; symbol Conn_01x06 -> Connector_Generic:Conn_01x06
- R1, R2, R3, R4: footprint Resistors_SMD:R_0805 -> Resistor_SMD:R_0805_2012Metric; symbol R -> Device:R
- U1: footprint TO_SOT_Packages_SMD:TSOT-23-5 -> Package_TO_SOT_SMD:SOT-23-5; symbol SPX3819 -> device.farm:SPX3819
- U2: footprint Housings_QFP:LQFP-32_7x7mm_Pitch0.8mm -> Package_QFP:LQFP-32_7x7mm_P0.8mm; symbol STM32F042K4Tx -> MCU_ST_STM32F0:STM32F042K4Tx
- X1: symbol I2C-6P -> device.farm:I2C-6P
- X2: symbol I2C -> device.farm:I2C
- X3: symbol SWD -> device.farm:SWD
