File: board/USB-I2C.sch (KiCad schematic (older format))
At the start: 17 parts, among them J1 USB_OTG, J2 Conn_01x06, U1 SPX3819, U2 STM32F042K4Tx, X1 I2C-6P, X2 I2C, X3 SWD

Commit message: WIP
Parts:
- removed C4, C5: 100n, Capacitor_SMD:C_0805_2012Metric, symbol Device:C
- removed U2: STM32F042K4Tx, Package_QFP:LQFP-32_7x7mm_P0.8mm, symbol MCU_ST_STM32F0:STM32F042K4Tx
- added U2: ATSAMD11C14A-SS, Package_SO:SOIC-14_3.9x8.7mm_P1.27mm, symbol MCU_Microchip_SAMD:ATSAMD11C14A-SS
Connections:
- net +3V3: now also U2.12 (VDD)
- net ALERT: now also U2.1 (PA05)
- net GND: now also U2.11 (GND)
- net SCL: now also U2.4 (PA14)
- net SDA: now also U2.5 (PA15)
- net SWCLK: now also U2.7 (PA30/SWCLK)
- net SWDIO: now also U2.8 (PA31/SWDIO)
- net USB_DM: now also U2.9 (PA24)
- net USB_DP: now also U2.10 (PA25)
- net LED: now reaches R1.1
- net LED: now also U2.13 (PA02)
- net at C1.1: now also U2.6 (PA28/~RST)
- no-connect marks 19 -> 5
Other:
- moved on the sheet: C1, C3, D1, R1, R2, R3, R4

Commit message: WIP
Parts:
- added J3: Conn_01x06, Connector_IDC:IDC-Header_2x03_P2.54mm_Vertical, symbol Connector_Generic:Conn_01x06
Connections:
- net +3V3: now also J3.4 (Pin_4)
- net +5V: now also J3.5 (Pin_5)
- net ALERT: now also J3.6 (Pin_6)
- net GND: now also J3.1 (Pin_1)
- net SCL: now also U2.5 (PA15), J3.2 (Pin_2); no longer U2.4 (PA14)
- net SDA: now also U2.4 (PA14), J3.3 (Pin_3); no longer U2.5 (PA15)
Changed lines of the file:
@@
 	1    0    0    -1
 $EndComp
+Text Label 6600 4450 0    60   ~ 0
+SCL
 Text Label 6600 4350 0    60   ~ 0
-SCL
-Text Label 6600 4450 0    60   ~ 0
 SDA
 Wire Wire Line
@@
 	0    1    1    0
 $EndComp
+$Comp
+L Connector_Generic:Conn_01x06 J3
+U 1 1 605F4A2B
+P 4400 6650
+F 0 "J3" H 4400 6950 50  0000 C CNN
+F 1 "Conn_01x06" H 4400 6250 50  0000 C CNN
+F 2 "Connector_IDC:IDC-Header_2x03_P2.54mm_Vertical" H 4400 6650 50  0001 C CNN
+F 3 "" H 4400 6650 50  0001 C CNN
+	1    4400 6650
+	-1   0    0    1
+$EndComp
+$Comp
+L power:+3.3V #PWR011
+U 1 1 605F4A35
+P 4600 6550
+F 0 "#PWR011" H 4600 6400 50  0001 C CNN
+F 1 "+3V3" V 4600 6750 50  0000 C CNN
+F 2 "" H 4600 6550 50  0001 C CNN
+F 3 "" H 4600 6550 50  0001 C CNN
+	1    4600 6550
+	0    1    1    0
+$EndComp
+$Comp
+L power:+5V #PWR010
+U 1 1 605F4A3F
+P 4600 6450
+F 0 "#PWR010" H 4600 6300 50  0001 C CNN
+F 1 "+5V" V 4600 6650 50  0000 C CNN
+F 2 "" H 4600 6450 50  0001 C CNN
+F 3 "" H 4600 6450 50  0001 C CNN
+	1    4600 6450
+	0    1    1    0
+$EndComp
+Text Label 4600 6350 0    60   ~ 0
+ALERT
+Text Label 4600 6650 0    60   ~ 0
+SDA
+Text Label 4600 6750 0    60   ~ 0
+SCL
+$Comp
+L power:GND #PWR012
+U 1 1 605F4A4C
+P 4600 6850
+F 0 "#PWR012" H 4600 6600 50  0001 C CNN
+F 1 "GND" V 4600 6650 50  0000 C CNN
+F 2 "" H 4600 6850 50  0001 C CNN
+F 3 "" H 4600 6850 50  0001 C CNN
+	1    4600 6850
+	0    -1   -1   0
+$EndComp
 $EndSCHEMATC
