File: board/USB-I2C.kicad_sch (KiCad schematic)
At the start: 16 parts, among them J1 USB_OTG, J2 Conn_01x06, J3 Conn_01x06, U1 SPX3819, U2 ATSAMD11C14A-SS, X1 I2C-6P, X2 I2C, X3 SWD

Commit message: WIP
Parts:
- removed C3: 100n, Capacitor_SMD:C_0805_2012Metric, symbol Device:C
- removed J1: USB_OTG, Drake:conn_usb_B_micro_smd-2, symbol Connector:USB_OTG
- removed U1: SPX3819, Package_TO_SOT_SMD:SOT-23-5, symbol Drake:SPX3819
- removed U2: ATSAMD11C14A-SS, Package_SO:SOIC-14_3.9x8.7mm_P1.27mm, symbol MCU_Microchip_SAMD:ATSAMD11C14A-SS
- removed X3: SWD, Drake:SWD, symbol Drake:SWD
- added C1: 10u, Capacitor_SMD:C_0805_2012Metric, symbol Device:C
- added C4, C5, C6: 100n, Capacitor_SMD:C_0805_2012Metric, symbol Device:C
- added C7: 1u, Capacitor_SMD:C_0805_2012Metric, symbol Device:C
- added C8, C9: 15p, Capacitor_SMD:C_0805_2012Metric, symbol Device:C
- added J4: USB_C_Receptacle, Connector_USB:USB_C_Receptacle_G-Switch_GT-USB-7010ASV, symbol Connector:USB_C_Receptacle
- added R5: 10k, Resistor_SMD:R_0805_2012Metric, symbol Device:R
- added R6: 1M, Resistor_SMD:R_0805_2012Metric, symbol Device:R
- added R7, R8: 5.11k 1%, Resistor_SMD:R_0805_2012Metric, symbol Device:R
- added U1: LM1117MP-3.3, Package_TO_SOT_SMD:SOT-223-3_TabPin2, symbol Regulator_Linear:LM1117MP-3.3
- added U2: ESP32-C3, Package_DFN_QFN:QFN-32-1EP_5x5mm_P0.5mm_EP3.45x3.45mm, symbol Espressif:ESP32-C3
- added Y1: 40MHz, Crystal:Crystal_SMD_3225-4Pin_3.2x2.5mm, symbol Device:Crystal_GND24_Small
- C2: value 1u -> 10u
- renumbered C1 to C3, J2 to J1
Connections:
- net +3V3: now also C3.1, C4.1, C5.1, C6.1, R5.2, U1.2 (VO), U2.11 (VDD3P3_RTC), U2.17 (VDD3P3_CPU), U2.2 (VDD3P3), U2.3 (VDD3P3), U2.31 (VDDA), U2.32 (VDDA)
- net +5V: now also C1.1, J4.A4 (VBUS), J4.A9 (VBUS), J4.B4 (VBUS), J4.B9 (VBUS), U1.3 (VI)
- net ALERT: now also U2.12 (MTCK/GPIO6)
- net GND: now also C1.2, C4.2, C5.2, C6.2, C7.1, C8.1, C9.1, J4.A1 (GND), J4.A12 (GND), J4.B1 (GND), J4.B12 (GND), R6.1, R7.2, R8.2, U1.1 (GND), U2.33 (GND), Y1.2, Y1.4
- net LED: now also U2.13 (MTDO/GPIO7)
- net SCL: now also U2.10 (MTDI/GPIO5/ADC2_CH0)
- net SDA: now also U2.9 (MTMS/GPIO4/ADC1_CH4)
- net USB_DM: now also J4.A7 (D-), J4.B7 (D-), U2.25 (GPIO18/USB_D-)
- net USB_DP: now also J4.A6 (D+), J4.B6 (D+), U2.26 (GPIO19/USB_D+)
- new net: J4.A5 (CC1), R7.1
- new net: J4.B5 (CC2), R8.1
- new net: J4.S1 (SHIELD), R6.2
- new net: C9.2, U2.30 (XTAL_P), Y1.1
- new net: C8.2, U2.29 (XTAL_N), Y1.3
- new net: C7.2, R5.1, U2.7 (CHIP_EN)
- no-connect marks 5 -> 27
Other:
- moved on the sheet: C3, D1, R1, R2, R3, R4

Commit message: WIP
Parts:
- U2: value ESP32-C3 -> ESP32-C3FN4
Changed lines of the file:
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@@
       (effects (font (size 1.27 1.27)))
     )
-    (property "Value" "ESP32-C3" (at 182.88 85.3981 0)
+    (property "Value" "ESP32-C3FN4" (at 182.88 85.3981 0)
       (effects (font (size 1.27 1.27)))
     )
